Commit message: refactor

File: assets/urdf/Diana/diana_v2.urdf (robot description, URDF)
Before this commit: robot diana_v2, 8 links, 7 joints
Links:
- link base: geometry collision mesh filename=/home/soumya_mondal/Desktop/Projects/Thesis/assets/urdf/Dia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; visual mesh filename=/home/soumya_mondal/Desktop/Projects/Thesis/assets/urdf/Dia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
- link link_1: geometry collision mesh filename=/home/soumya_mondal/Desktop/Projects/Thesis/assets/urdf/Dia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; visual mesh filename=/home/soumya_mondal/Desktop/Projects/Thesis/assets/urdf/Dia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
- link link_2: geometry collision mesh filename=/home/soumya_mondal/Desktop/Projects/Thesis/assets/urdf/Dia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; visual mesh filename=/home/soumya_mondal/Desktop/Projects/Thesis/assets/urdf/Dia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
- link link_3: geometry collision mesh filename=/home/soumya_mondal/Desktop/Projects/Thesis/assets/urdf/Dia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; visual mesh filename=/home/soumya_mondal/Desktop/Projects/Thesis/assets/urdf/Dia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
- link link_4: geometry collision mesh filename=/home/soumya_mondal/Desktop/Projects/Thesis/assets/urdf/Dia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; visual mesh filename=/home/soumya_mondal/Desktop/Projects/Thesis/assets/urdf/Dia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
- link link_5: geometry collision mesh filename=/home/soumya_mondal/Desktop/Projects/Thesis/assets/urdf/Dia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; visual mesh filename=/home/soumya_mondal/Desktop/Projects/Thesis/assets/urdf/Dia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
- link link_6: geometry collision mesh filename=/home/soumya_mondal/Desktop/Projects/Thesis/assets/urdf/Dia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; visual mesh filename=/home/soumya_mondal/Desktop/Projects/Thesis/assets/urdf/Dia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
- link link_7: geometry collision mesh filename=/home/soumya_mondal/Desktop/Projects/Thesis/assets/urdf/Dia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; visual mesh filename=/home/soumya_mondal/Desktop/Projects/Thesis/assets/urdf/Dia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
